Commit message: made aliengo walk

File: resources/robots/aliengo/urdf/aliengo.urdf (robot description, URDF)
Before this commit: robot aliengo, 31 links, 30 joints
Links:
- removed link FL_calf_rotor
- removed link FL_hip_rotor
- removed link FL_thigh_rotor
- removed link FR_calf_rotor
- removed link FR_hip_rotor
- removed link FR_thigh_rotor
- removed link RL_calf_rotor
- removed link RL_hip_rotor
- removed link RL_thigh_rotor
- removed link RR_calf_rotor
- removed link RR_hip_rotor
- removed link RR_thigh_rotor
- removed link trunk
- link base: mass None -> 11.644; geometry collision box size=0.647 0.15 0.112; visual mesh filename=../dae/trunk.dae scale=1 1 1
Joints:
- removed joint FL_calf_rotor_joint
- removed joint FL_foot_fixed
- removed joint FL_hip_rotor_joint
- removed joint FL_thigh_rotor_joint
- removed joint FR_calf_rotor_joint
- removed joint FR_foot_fixed
- removed joint FR_hip_rotor_joint
- removed joint FR_thigh_rotor_joint
- removed joint RL_calf_rotor_joint
- removed joint RL_foot_fixed
- removed joint RL_hip_rotor_joint
- removed joint RL_thigh_rotor_joint
- removed joint RR_calf_rotor_joint
- removed joint RR_foot_fixed
- removed joint RR_hip_rotor_joint
- removed joint RR_thigh_rotor_joint
- removed joint floating_base
- added joint FL_foot_joint: type fixed, parent FL_calf, child FL_foot, origin xyz=0 0 -0.25 rpy=0 0 0
- added joint FR_foot_joint: type fixed, parent FR_calf, child FR_foot, origin xyz=0 0 -0.25 rpy=0 0 0
- added joint RL_foot_joint: type fixed, parent RL_calf, child RL_foot, origin xyz=0 0 -0.25 rpy=0 0 0
- added joint RR_foot_joint: type fixed, parent RR_calf, child RR_foot, origin xyz=0 0 -0.25 rpy=0 0 0
- joint FL_hip_joint: parent trunk -> base
- joint FL_thigh_joint: type continuous -> revolute
- joint FR_hip_joint: parent trunk -> base
- joint FR_thigh_joint: type continuous -> revolute
- joint RL_hip_joint: parent trunk -> base
- joint RL_thigh_joint: type continuous -> revolute
- joint RR_hip_joint: parent trunk -> base
- joint RR_thigh_joint: type continuous -> revolute
- joint imu_joint: parent trunk -> base
